Commit message: Fix Xacro File

File: go2w_description/urdf/const.xacro (robot description, xacro)
@@ -10,13 +10,14 @@
     <xacro:property name="head_upper_length" value="0.09"/>
     <xacro:property name="head_lower_radius" value="0.06"/>
+    <xacro:property name="hip_offset_col_y" value="0.08"/>
     <xacro:property name="hip_radius" value="0.046"/>
     <xacro:property name="hip_length" value="0.04"/>
-    <xacro:property name="thigh_offset_z" value="-0.1065"/>
-    <xacro:property name="thigh_length" value="0.032"/>
+    <xacro:property name="thigh_offset_col_z" value="-0.1065"/>
+    <xacro:property name="thigh_length" value="0.11"/>
     <xacro:property name="thigh_width" value="0.0245"/>
     <xacro:property name="thigh_height" value="0.034"/>
-    <xacro:property name="calf_offset_x" value="0.01"/>
-    <xacro:property name="calf_offset_z" value="-0.06"/>
-    <xacro:property name="calf_rotation_p" value="-0.2"/>
+    <xacro:property name="calf_offset_col_x" value="0.01"/>
+    <xacro:property name="calf_offset_col_z" value="-0.06"/>
+    <xacro:property name="calf_rotation_col_p" value="-0.2"/>
     <xacro:property name="calf_length" value="0.12"/>
     <xacro:property name="calf_radius" value="0.013"/>

File: go2w_description/urdf/go2w_description.urdf.xacro (robot description, xacro)
@@ -43,5 +43,5 @@
       </visual>
       <collision>
-        <origin rpy="${PI/2.0} 0 0" xyz="0 0.08 0" />
+        <origin rpy="${PI/2.0} 0 0" xyz="0 ${hip_offset_col_y*left_sign} 0" />
         <geometry>
             <cylinder length="${hip_length}" radius="${hip_radius}" />
@@ -81,5 +81,5 @@
       </visual>
       <collision>
-        <origin rpy="0 ${PI/2.0} 0" xyz="0 0 ${thigh_offset_z}" />
+        <origin rpy="0 ${PI/2.0} 0" xyz="0 0 ${thigh_offset_col_z}" />
         <geometry>
           <box size="${thigh_length} ${thigh_width} ${thigh_height}" />
@@ -116,5 +116,5 @@
       </visual>
       <collision>
-        <origin rpy="0 ${calf_rotation_p} 0" xyz="${calf_offset_x} 0 ${calf_offset_z}" />
+        <origin rpy="0 ${calf_rotation_col_p} 0" xyz="${calf_offset_col_x} 0 ${calf_offset_col_z}" />
         <geometry>
           <cylinder length="${calf_length}" radius="${calf_radius}" />

Commit message: Champ (High Level Walk) Implemented

File: go2w_description/urdf/const.xacro (robot description, xacro)
@@ -28,4 +28,7 @@
     <xacro:property name="foot_motor_length" value="0.05"/>
     <xacro:property name="foot_motor_radius" value="0.05"/>
+    <xacro:property name="foot_offset_col_y" value="0.05"/>
+    <xacro:property name="foot_length" value="0.05"/>
+    <xacro:property name="foot_radius" value="0.085"/>
     <!-- offset of link locations -->
     <xacro:property name="hip_offset_x" value="0.1934"/>
@@ -53,18 +56,22 @@
     <xacro:property name="foot_offset_z" value="-0.2264"/>
     <!-- joint limits -->
-    <!-- <xacro:property name="damping" value="0.01"/>
-    <xacro:property name="friction" value="0.2"/> -->
     <xacro:property name="hip_position_max" value="1.0472"/>
     <xacro:property name="hip_position_min" value="-1.0472"/>
     <xacro:property name="hip_velocity_max" value="30.1"/>
     <xacro:property name="hip_torque_max" value="23.7"/>
+    <xacro:property name="hip_damping" value="0.1"/>
+    <xacro:property name="hip_friction" value="0.2"/>
     <xacro:property name="thigh_position_max" value="3.4907"/>
     <xacro:property name="thigh_position_min" value="-1.5708"/>
     <xacro:property name="thigh_velocity_max" value="30.1"/>
     <xacro:property name="thigh_torque_max" value="23.7"/>
+    <xacro:property name="thigh_damping" value="0.1"/>
+    <xacro:property name="thigh_friction" value="0.2"/>
     <xacro:property name="calf_position_max" value="-0.83776"/>
     <xacro:property name="calf_position_min" value="-2.7227"/>
     <xacro:property name="calf_velocity_max" value="20.06"/>
     <xacro:property name="calf_torque_max" value="35.55"/>
+    <xacro:property name="calf_damping" value="0.1"/>
+    <xacro:property name="calf_friction" value="0.2"/>
     <xacro:property name="foot_velocity_max" value="30.1"/>
     <xacro:property name="foot_torque_max" value="23.7"/>

File: go2w_description/urdf/go2w_description.urdf.xacro (robot description, xacro)
@@ -60,4 +60,5 @@
         <limit effort="${hip_torque_max}" velocity="${hip_velocity_max}" lower="${-hip_position_max}" upper="${-hip_position_min}"/>
       </xacro:if>
+      <dynamics damping="${hip_damping}" friction="${hip_friction}" />
     </joint>
     <!-- Thigh -->
@@ -93,4 +94,5 @@
       <axis xyz="0 1 0" />
       <limit effort="${thigh_torque_max}" velocity="${thigh_velocity_max}" lower="${thigh_position_min}" upper="${thigh_position_max}" />
+      <dynamics damping="${thigh_damping}" friction="${thigh_friction}" />
     </joint>
     <!-- Calf -->
@@ -128,4 +130,5 @@
       <axis xyz="0 1 0" />
       <limit lower="${calf_position_min}" upper="${calf_position_max}" effort="${calf_torque_max}" velocity="${calf_velocity_max}" />
+      <dynamics damping="${calf_damping}" friction="${calf_friction}" />
     </joint>
     <!-- Calf lower -->
@@ -201,21 +204,16 @@
       </visual>
       <collision>
-        <origin rpy="0 0 0" xyz="0 0.0 0" />
-        <geometry>
-          <xacro:if value="${left == True}">
-            <mesh filename="${mesh_prefix}/left_wheel.dae" />
-            </xacro:if>
-            <xacro:if value="${left == False}">
-            <mesh filename="${mesh_prefix}/right_wheel.dae" />
-            </xacro:if>
-        </geometry>
-      </collision>
-    </link>
-    <joint name="${prefix}_foot_joint" type="continuous">
+        <origin rpy="${PI/2.0} 0 0" xyz="0 ${foot_offset_col_y*left_sign} 0" />
+        <geometry>
+          <cylinder length="${foot_length}" radius="${foot_radius}" />
+        </geometry>
+      </collision>
+    </link>
+    <joint name="${prefix}_foot_joint" type="fixed">
       <origin xyz="${foot_offset_x} ${foot_offset_y*left_sign} ${foot_offset_z}" rpy="0 0 0" />
       <parent link="${prefix}_calf" />
       <child link="${prefix}_foot" />
       <axis xyz="0 1 0" />
-        <limit effort="${foot_torque_max}" velocity="${foot_velocity_max}" />
+      <!-- <limit effort="${foot_torque_max}" velocity="${foot_velocity_max}" /> -->
     </joint>
     <!-- Gazebo ros2_control -->
@@ -226,6 +224,6 @@
       <joint name="${prefix}_hip_joint">
         <command_interface name="effort">
-          <!-- <param name="min">${hip_torque_min}</param>
-          <param name="max">${hip_torque_max}</param> -->
+          <param name="min">${-hip_torque_max}</param>
+          <param name="max">${hip_torque_max}</param>
         </command_interface>
         <state_interface name="position">
@@ -233,10 +231,10 @@
         </state_interface>
         <state_interface name="velocity"/>
-        <!-- <state_interface name="effort"/> -->
+        <state_interface name="effort"/>
       </joint>
       <joint name="${prefix}_thigh_joint">
         <command_interface name="effort">
-          <!-- <param name="min">${thigh_torque_min}</param>
-          <param name="max">${thigh_torque_max}</param> -->
+          <param name="min">${-thigh_torque_max}</param>
+          <param name="max">${thigh_torque_max}</param>
         </command_interface>
         <state_interface name="position">
@@ -244,10 +242,10 @@
         </state_interface>
         <state_interface name="velocity"/>
-        <!-- <state_interface name="effort"/> -->
+        <state_interface name="effort"/>
       </joint>
       <joint name="${prefix}_calf_joint">
         <command_interface name="effort">
-          <!-- <param name="min">${calf_torque_min}</param>
-          <param name="max">${calf_torque_max}</param> -->
+          <param name="min">${-calf_torque_max}</param>
+          <param name="max">${calf_torque_max}</param>
         </command_interface>
         <state_interface name="position">
@@ -255,10 +253,10 @@
         </state_interface>
         <state_interface name="velocity"/>
-        <!-- <state_interface name="effort"/> -->
+        <state_interface name="effort"/>
       </joint>
       <joint name="${prefix}_foot_joint">
         <command_interface name="velocity">
-          <!-- <param name="min">-100.0</param>
-          <param name="max">100.0</param> -->
+          <param name="min">${-foot_velocity_max}</param>
+          <param name="max">${foot_velocity_max}</param>
         </command_interface>
         <state_interface name="position">
@@ -268,5 +266,5 @@
           <param name="initial_value">0.0</param>
         </state_interface>
-        <!-- <state_interface name="effort"/> -->
+        <state_interface name="effort"/>
       </joint>
     </ros2_control>

Commit message: High-Level linear motions and angular rotation OK

File: go2w_description/urdf/const.xacro (robot description, xacro)
@@ -4,7 +4,7 @@
     <xacro:property name="PI" value="3.1415926535897931"/>
     <!-- simplified collision value -->
-    <xacro:property name="base_width" value="0.0935"/>
-    <xacro:property name="base_length" value="0.3762"/>
-    <xacro:property name="base_width" value="0.114"/>
+    <xacro:property name="body_width" value="0.0935"/>
+    <xacro:property name="body_length" value="0.3762"/>
+    <xacro:property name="body_width" value="0.114"/>
     <xacro:property name="head_upper_radius" value="0.06"/>
     <xacro:property name="head_upper_length" value="0.09"/>
@@ -81,15 +81,15 @@
     <xacro:property name="calf_init_position" value="-2.0287070274353027"/>
     <!-- dynamics inertial value -->
-    <!-- base -->
-    <xacro:property name="base_mass" value="6.921"/>
-    <xacro:property name="base_com_x" value="0.021112"/>
-    <xacro:property name="base_com_y" value="0.00"/>
-    <xacro:property name="base_com_z" value="-0.005366"/>
-    <xacro:property name="base_ixx" value="0.02448"/>
-    <xacro:property name="base_ixy" value="0.00012166"/>
-    <xacro:property name="base_ixz" value="0.0014849"/>
-    <xacro:property name="base_iyy" value="0.098077"/>
-    <xacro:property name="base_iyz" value="-3.12E-05"/>
-    <xacro:property name="base_izz" value="0.107"/>
+    <!-- body -->
+    <xacro:property name="body_mass" value="6.921"/>
+    <xacro:property name="body_com_x" value="0.021112"/>
+    <xacro:property name="body_com_y" value="0.00"/>
+    <xacro:property name="body_com_z" value="-0.005366"/>
+    <xacro:property name="body_ixx" value="0.02448"/>
+    <xacro:property name="body_ixy" value="0.00012166"/>
+    <xacro:property name="body_ixz" value="0.0014849"/>
+    <xacro:property name="body_iyy" value="0.098077"/>
+    <xacro:property name="body_iyz" value="-3.12E-05"/>
+    <xacro:property name="body_izz" value="0.107"/>
     <!-- head upper -->
     <xacro:property name="head_upper_mass" value="0.001"/>

File: go2w_description/urdf/go2w_description.urdf.xacro (robot description, xacro)
@@ -51,5 +51,5 @@
     <joint name="${prefix}_hip_joint" type="revolute">
       <origin xyz="${hip_offset_x*front_sign} ${hip_offset_y*left_sign} ${hip_offset_z}" rpy="0 0 0" />
-      <parent link="base" />
+      <parent link="body" />
       <child link="${prefix}_hip" />
       <axis xyz="1 0 0" />
@@ -210,16 +210,175 @@
       </collision>
     </link>
-    <joint name="${prefix}_foot_joint" type="fixed">
+    <joint name="${prefix}_foot_joint" type="continuous">
       <origin xyz="${foot_offset_x} ${foot_offset_y*left_sign} ${foot_offset_z}" rpy="0 0 0" />
       <parent link="${prefix}_calf" />
       <child link="${prefix}_foot" />
       <axis xyz="0 1 0" />
-      <!-- <limit effort="${foot_torque_max}" velocity="${foot_velocity_max}" /> -->
-    </joint>
-    <!-- Gazebo ros2_control -->
-    <ros2_control name="${prefix}" type="system">
-      <hardware>
-      <plugin>gazebo_ros2_control/GazeboSystem</plugin>
-      </hardware>
+      <limit effort="${foot_torque_max}" velocity="${foot_velocity_max}" />
+    </joint>
+    <gazebo reference="${prefix}_foot">
+        <mu1>3</mu1>
+        <mu2>3</mu2>
+    </gazebo>
+  </xacro:macro>
+  <!-- Base-->
+  <link name="base"/>
+  <!-- Body -->
+  <link name="body">
+    <inertial>
+      <origin xyz="${body_com_x} ${body_com_y} ${body_com_z}" rpy="0 0 0" />
+      <mass value="${body_mass}" />
+      <inertia ixx="${body_ixx}" ixy="${body_ixy}" ixz="${body_ixz}" iyy="${body_iyy}" iyz="${body_iyz}" izz="${body_izz}" />
+    </inertial>
+    <visual>
+      <origin xyz="0 0 0" rpy="0 0 0" />
+      <geometry>
+        <mesh filename="${mesh_prefix}/base.dae" />
+      </geometry>
+      <material name="深色橡胶_001-effect"><color rgba="0.6717055 0.6924257 0.7742702 1" /></material><material name="白色logo_001-effect"><color rgba="1 1 1 1" /></material><material name="黑色贴纸_007-effect"><color rgba="0.009018 0.009018 0.009018 1" /></material><material name="黑色金属_007-effect"><color rgba="0.01341 0.01341 0.01341 1" /></material><material name="黑色塑料_003-effect"><color rgba="0.023455 0.023455 0.023455 1" /></material></visual>
+    <collision>
+      <origin rpy="0 0 0" xyz="0 0 0" />
+      <geometry>
+        <box size="${body_length} ${body_width} ${body_width}" />
+      </geometry>
+    </collision>
+  </link>
+  <joint name="body_joint" type="fixed">
+    <parent link="base" />
+    <child link="body" />
+  </joint>
+  <!-- Head Upper-->
+  <link name="Head_upper">
+    <inertial>
+      <origin xyz="${head_upper_com_x} ${head_upper_com_y} ${head_upper_com_z}" rpy="0 0 0" />
+      <mass value="${head_upper_mass}" />
+      <inertia ixx="${head_upper_ixx}" ixy="${head_upper_ixy}" ixz="${head_upper_ixz}" iyy="${head_upper_iyy}" iyz="${head_upper_iyz}" izz="${head_upper_izz}" />
+    </inertial>
+    <collision>
+      <origin xyz="0 0 0" rpy="0 0 0" />
+      <geometry>
+        <cylinder radius="${head_upper_radius}" length="${head_upper_length}" />
+      </geometry>
+    </collision>
+  </link>
+  <joint name="Head_upper_joint" type="fixed" dont_collapse="true">
+    <origin xyz="0.285 0 0.01" rpy="0 0 0" />
+    <parent link="body" />
+    <child link="Head_upper" />
+    <axis xyz="0 0 0" />
+  </joint>
+  <!-- Head Lower -->
+  <link name="Head_lower">
+    <inertial>
+      <origin xyz="${head_lower_com_x} ${head_lower_com_y} ${head_lower_com_z}" rpy="0 0 0" />
+      <mass value="${head_lower_mass}" />
+      <inertia ixx="${head_lower_ixx}" ixy="${head_lower_ixy}" ixz="${head_lower_ixz}" iyy="${head_lower_iyy}" iyz="${head_lower_iyz}" izz="${head_lower_izz}" />
+    </inertial>
+    <collision>
+      <origin xyz="0 0 0" rpy="0 0 0" />
+      <geometry>
+        <sphere radius="${head_lower_radius}" />
+      </geometry>
+    </collision>
+  </link>
+  <joint name="Head_lower_joint" type="fixed" dont_collapse="true">
+    <origin xyz="0.008 0 -0.07" rpy="0 0 0" />
+    <parent link="Head_upper" />
+    <child link="Head_lower" />
+    <axis xyz="0 0 0" />
+  </joint>
+  <xacro:leg prefix="FL" front="True" left="True"/>
+  <xacro:leg prefix="FR" front="True" left="False"/>
+  <xacro:leg prefix="RL" front="False" left="True"/>
+  <xacro:leg prefix="RR" front="False" left="False"/>
+  <!-- IMU -->
+  <link name="imu">
+    <inertial>
+      <origin xyz="0 0 0" rpy="0 0 0" />
+      <mass value="0" />
+      <inertia ixx="0" ixy="0" ixz="0" iyy="0" iyz="0" izz="0" />
+    </inertial>
+  </link>
+  <joint name="imu_joint" type="fixed">
+    <origin xyz="-0.02557 0 0.04232" rpy="0 0 0" />
+    <parent link="body" />
+    <child link="imu" />
+    <axis xyz="0 0 0" />
+  </joint>
+  <gazebo reference="imu">
+    <sensor name="imu_sensor" type="imu">
+      <always_on>true</always_on>
+      <update_rate>100</update_rate>
+      <imu>
+        <angular_velocity>
+          <x>
+            <noise type="gaussian">
+              <mean>0.0</mean>
+              <stddev>2e-4</stddev>
+            </noise>
+          </x>
+          <y>
+            <noise type="gaussian">
+              <mean>0.0</mean>
+              <stddev>2e-4</stddev>
+            </noise>
+          </y>
+          <z>
+            <noise type="gaussian">
+              <mean>0.0</mean>
+              <stddev>2e-4</stddev>
+            </noise>
+          </z>
+        </angular_velocity>
+        <linear_acceleration>
+            <x>
+              <noise type="gaussian">
+                <mean>0.0</mean>
+                <stddev>1.7e-2</stddev>
+              </noise>
+            </x>
+            <y>
+              <noise type="gaussian">
+                <mean>0.0</mean>
+                <stddev>1.7e-2</stddev>
+              </noise>
+            </y>
+            <z>
+              <noise type="gaussian">
+                <mean>0.0</mean>
+                <stddev>1.7e-2</stddev>
+              </noise>
+            </z>
+        </linear_acceleration>
+      </imu>
+      <plugin name="imu_plugin" filename="libgazebo_ros_imu_sensor.so">
+        <ros>
+          <namespace>imu</namespace>
+          <remapping>~/out:=data</remapping>
+        </ros>
+        <initial_orientation_as_reference>false</initial_orientation_as_reference>
+      </plugin>
+    </sensor>
+  </gazebo>
+  <!-- Radar -->
+  <link name="radar">
+    <inertial>
+      <origin xyz="0 0 0" rpy="0 0 0" />
+      <mass value="0" />
+      <inertia ixx="0" ixy="0" ixz="0" iyy="0" iyz="0" izz="0" />
+    </inertial>
+  </link>
+  <joint name="radar_joint" type="fixed">
+    <origin xyz="0.28945 0 -0.046825" rpy="0 2.8782 0" />
+    <parent link="body" />
+    <child link="radar" />
+    <axis xyz="0 0 0" />
+  </joint>
+  <!-- Gazebo ros2_control -->
+  <ros2_control name="gazebo_ros2_control" type="system">
+    <hardware>
+    <plugin>gazebo_ros2_control/GazeboSystem</plugin>
+    </hardware>
+    <xacro:macro name="joint_ros2_control" params="prefix">
       <joint name="${prefix}_hip_joint">
         <command_interface name="effort">
@@ -268,95 +427,13 @@
         <state_interface name="effort"/>
       </joint>
-    </ros2_control>
-  </xacro:macro>
-  <link name="base">
-    <inertial>
-      <origin xyz="${base_com_x} ${base_com_y} ${base_com_z}" rpy="0 0 0" />
-      <mass value="${base_mass}" />
-      <inertia ixx="${base_ixx}" ixy="${base_ixy}" ixz="${base_ixz}" iyy="${base_iyy}" iyz="${base_iyz}" izz="${base_izz}" />
-    </inertial>
-    <visual>
-      <origin xyz="0 0 0" rpy="0 0 0" />
-      <geometry>
-        <mesh filename="${mesh_prefix}/base.dae" />
-      </geometry>
-      <material name="深色橡胶_001-effect"><color rgba="0.6717055 0.6924257 0.7742702 1" /></material><material name="白色logo_001-effect"><color rgba="1 1 1 1" /></material><material name="黑色贴纸_007-effect"><color rgba="0.009018 0.009018 0.009018 1" /></material><material name="黑色金属_007-effect"><color rgba="0.01341 0.01341 0.01341 1" /></material><material name="黑色塑料_003-effect"><color rgba="0.023455 0.023455 0.023455 1" /></material></visual>
-    <collision>
-      <origin rpy="0 0 0" xyz="0 0 0" />
-      <geometry>
-        <box size="${base_length} ${base_width} ${base_width}" />
-      </geometry>
-    </collision>
-  </link>
-  <link name="Head_upper">
-    <inertial>
-      <origin xyz="${head_upper_com_x} ${head_upper_com_y} ${head_upper_com_z}" rpy="0 0 0" />
-      <mass value="${head_upper_mass}" />
-      <inertia ixx="${head_upper_ixx}" ixy="${head_upper_ixy}" ixz="${head_upper_ixz}" iyy="${head_upper_iyy}" iyz="${head_upper_iyz}" izz="${head_upper_izz}" />
-    </inertial>
-    <collision>
-      <origin xyz="0 0 0" rpy="0 0 0" />
-      <geometry>
-        <cylinder radius="${head_upper_radius}" length="${head_upper_length}" />
-      </geometry>
-    </collision>
-  </link>
-  <joint name="Head_upper_joint" type="fixed" dont_collapse="true">
-    <origin xyz="0.285 0 0.01" rpy="0 0 0" />
-    <parent link="base" />
-    <child link="Head_upper" />
-    <axis xyz="0 0 0" />
-  </joint>
-  <link name="Head_lower">
-    <inertial>
-      <origin xyz="${head_lower_com_x} ${head_lower_com_y} ${head_lower_com_z}" rpy="0 0 0" />
-      <mass value="${head_lower_mass}" />
-      <inertia ixx="${head_lower_ixx}" ixy="${head_lower_ixy}" ixz="${head_lower_ixz}" iyy="${head_lower_iyy}" iyz="${head_lower_iyz}" izz="${head_lower_izz}" />
-    </inertial>
-    <collision>
-      <origin xyz="0 0 0" rpy="0 0 0" />
-      <geometry>
-        <sphere radius="${head_lower_radius}" />
-      </geometry>
-    </collision>
-  </link>
-  <joint name="Head_lower_joint" type="fixed" dont_collapse="true">
-    <origin xyz="0.008 0 -0.07" rpy="0 0 0" />
-    <parent link="Head_upper" />
-    <child link="Head_lower" />
-    <axis xyz="0 0 0" />
-  </joint>
-  <xacro:leg prefix="FL" front="True" left="True"/>
-  <xacro:leg prefix="FR" front="True" left="False"/>
-  <xacro:leg prefix="RL" front="False" left="True"/>
-  <xacro:leg prefix="RR" front="False" left="False"/>
-  <link name="imu">
-    <inertial>
-      <origin xyz="0 0 0" rpy="0 0 0" />
-      <mass value="0" />
-      <inertia ixx="0" ixy="0" ixz="0" iyy="0" iyz="0" izz="0" />
-    </inertial>
-  </link>
-  <joint name="imu_joint" type="fixed">
-    <origin xyz="-0.02557 0 0.04232" rpy="0 0 0" />
-    <parent link="base" />
-    <child link="imu" />
-    <axis xyz="0 0 0" />
-  </joint>
-  <link name="radar">
-    <inertial>
-      <origin xyz="0 0 0" rpy="0 0 0" />
-      <mass value="0" />
-      <inertia ixx="0" ixy="0" ixz="0" iyy="0" iyz="0" izz="0" />
-    </inertial>
-  </link>
-  <joint name="radar_joint" type="fixed">
-    <origin xyz="0.28945 0 -0.046825" rpy="0 2.8782 0" />
-    <parent link="base" />
-    <child link="radar" />
-    <axis xyz="0 0 0" />
-  </joint>
+    </xacro:macro>
+    <xacro:joint_ros2_control prefix="FL"/>
+    <xacro:joint_ros2_control prefix="FR"/>
+    <xacro:joint_ros2_control prefix="RL"/>
+    <xacro:joint_ros2_control prefix="RR"/>
+  </ros2_control>
+  <!-- Gazebo plugin for ros2_control -->
   <gazebo>
-      <plugin filename="libgazebo_ros2_control.so" name="gazebo_ros2_control">
+    <plugin filename="libgazebo_ros2_control.so" name="gazebo_ros2_control">
       <parameters>$(find go2w_description)/config/joint_controller.yaml</parameters>
     </plugin>
